Commit message: Robot vertical adjust

File: catkin_ws/src/my_robot/urdf/my_robot.xacro (robot description, xacro)
@@ -4,5 +4,5 @@
   <link name="robot_footprint"></link>
   <joint name="robot_footprint_joint" type="fixed">
-    <origin xyz="0 0 0" rpy="0 0 0" />
+    <origin xyz="0 0 0.2" rpy="0 0 0" />
     <parent link="robot_footprint"/>
     <child link="chassis" />

Commit message: final adjust

File: catkin_ws/src/my_robot/urdf/my_robot.xacro (robot description, xacro)
@@ -145,5 +145,5 @@
   </link>
   <joint type="fixed" name="hokuyo_joint">
-    <origin xyz="0.30 0 .1" rpy="0 0 0"/>
+    <origin xyz="0.38 0 .13" rpy="0 0 0"/>
     <child link="hokuyo"/>
     <parent link="chassis"/>
